File: Attenuverter/Attenuverter.kicad_pcb (KiCad board)
At the start: 2 copper layers, 30 x 100 mm, 49 parts, among them J1 AudioJack2_SwitchT, J2 AudioJack2_SwitchT, J3 AudioJack2_SwitchT, J4 AudioJack2_SwitchT, J5 AudioJack2_SwitchT, J6 AudioJack2_SwitchT, J7 Conn_02x05_Odd_Even, J8 AudioJack2_SwitchT, J9 AudioJack2_SwitchT, U1 TL084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

Commit message: Finish routing
Parts:
- moved C4 13.7 mm to (121.2, 128.0)
- moved R11 13.7 mm to (116.4, 126.0)
- moved U2 13.7 mm to (120.8, 125.0)
- moved C7 5.35 mm to (102.5, 106.8), turned to 90 degrees
- moved C2 5.26 mm to (116.8, 101.8), turned to 270 degrees
- moved C1 4.19 mm to (102.5, 101.5), turned to 270 degrees
- moved C3 3.69 mm to (118.8, 101.8), turned to 90 degrees
- moved R6 3.45 mm to (114.8, 101.7), turned to 270 degrees
- moved R12 3.45 mm to (114.8, 106.7), turned to 90 degrees
- moved R17 0.56 mm to (105.8, 108.0)
- moved C5 0.50 mm to (104.2, 82.5)
- moved C8 0.50 mm to (112.8, 82.5)
- moved C9 0.35 mm to (110.5, 108.0)
- moved C6 0.25 mm to (110.2, 98.0)
- moved R1 0.25 mm to (105.7, 98.0)
Connections:
- J7 pad 3: Net-(J7-Pad3) -> GND
- J7 pad 4: Net-(J7-Pad3) -> GND
- J7 pad 5: Net-(J7-Pad3) -> GND
- J7 pad 6: Net-(J7-Pad3) -> GND
- J7 pad 7: Net-(J7-Pad3) -> GND
- J7 pad 8: Net-(J7-Pad3) -> GND
- RV1 pad : (no net) -> GND
- RV2 pad : (no net) -> GND
- RV3 pad : (no net) -> GND
- RV4 pad : (no net) -> GND
- U1 pad 13: GND -> Net-(R20-Pad1)
- U1 pad 2: GND -> Net-(R4-Pad1)
- U1 pad 6: GND -> Net-(R10-Pad2)
- U1 pad 9: GND -> Net-(R15-Pad1)
Routing:
- net +5V: track 0.00 -> 87.2 mm, vias 0 -> 3
- net +12V: track 0.00 -> 82.5 mm, vias 0 -> 2
- net Net-(C1-Pad2): track 0.00 -> 66.5 mm, vias 0 -> 2
- net -12V: track 0.00 -> 58.0 mm, vias 0 -> 2
- net Net-(C1-Pad1): track 0.00 -> 52.6 mm, vias 0 -> 2
- net Net-(R4-Pad1): track 0.00 -> 50.0 mm, vias 0 -> 1
- net Net-(C7-Pad1): track 0.00 -> 48.0 mm
- net Net-(C7-Pad2): track 0.00 -> 47.1 mm, vias 0 -> 2
- net Net-(R20-Pad1): track 0.00 -> 43.4 mm, vias 0 -> 2
- net Net-(J1-PadT): track 0.00 -> 35.3 mm
- net Net-(J8-PadT): track 0.00 -> 34.5 mm
- net Net-(C2-Pad2): track 0.00 -> 32.3 mm
- net Net-(J5-PadT): track 0.00 -> 29.5 mm
- net Net-(J3-PadT): track 0.00 -> 27.8 mm
- net Net-(C3-Pad2): track 0.00 -> 27.0 mm
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Other:
- net class Power added: clearance 0.2, trace_width 1, via_dia 1, via_drill 0.6

Commit message: Generate gerbers and step
Other:
- board text added: "Attenuverter v1.0"
- board text added: "schenktronics.com"

Commit message: Swap inverting and non inverting inputs.  Generate gerbers
Connections:
- U1 pad 10: Net-(C3-Pad2) -> Net-(R15-Pad1)
- U1 pad 12: Net-(C7-Pad2) -> Net-(R20-Pad1)
- U1 pad 13: Net-(R20-Pad1) -> Net-(C7-Pad2)
- U1 pad 2: Net-(R4-Pad1) -> Net-(C1-Pad2)
- U1 pad 3: Net-(C1-Pad2) -> Net-(R4-Pad1)
- U1 pad 5: Net-(C2-Pad2) -> Net-(R10-Pad2)
- U1 pad 6: Net-(R10-Pad2) -> Net-(C2-Pad2)
- U1 pad 9: Net-(R15-Pad1) -> Net-(C3-Pad2)
Routing:
- net Net-(C2-Pad2): track 32.3 -> 28.9 mm
- net Net-(C7-Pad2): track 47.1 -> 50.0 mm
- net Net-(C1-Pad2): track 66.5 -> 69.3 mm
- net Net-(R4-Pad1): track 50.0 -> 51.2 mm
- net Net-(R20-Pad1): track 43.4 -> 44.3 mm
- net Net-(C3-Pad2): track 27.0 -> 26.2 mm
Other:
- board text added: "-12v +12v"
- board text added: "Red Stripe"
