File: AttenuverterFaceplate/AttenuverterFaceplate.kicad_pcb (KiCad board)
At the start: 2 copper layers, 30 x 128.5 mm, 16 parts

Commit message: Finish faceplate
Parts:
- added G***: LOGO, _NTSFootprints:SchentronicsLogo, F.Cu at (130.2, 146.5)
Routing:
- added copper zone on F.Cu, net (none)
Other:
- board text added: "Attenuverter"
